File: DMFX-1/DMFX-1 v1.0.brd (EAGLE design)
At the start: 144 x 100 mm, 566 parts, among them IC2 SN74HC4066D, J1 USB-MINIB-5PIN, J1-2 USB-MINIB-5PIN, J10 MONOSW3C, J11 DM3BT-DSF-PEJS, J2 USB-B-SMT, J3 STEREOSW3C, J4 HEADPHONES, J5 87409-110LF, J6 DM3BT-DSF-PEJS, J7 87409-110LF, J8 DCJ0202, J9 MONOSW3C, Q1 MUN2214T1, Q10 MUN2214T1, Q2 MUN2214T1, Q3 MMBF4393, Q4 MUN2214T1, Q5 2N7002ET1G, Q6 2N7002ET1G, Q7 2N7002ET1G, Q8 MUN2214T1, Q9 MUN2214T1, SW1 MB2011SB1W03-DA, SW2 OS102011MA1Q, U10X 24C64SM, U11X TPS73201DBVT, U12X TPS562209SO, U13 741G3157DBVR, U14 ASDM1-12.000MHZ-LC-T, U15X CDCLVC1108PWR, U17 TLV320AIC3204IRHBT, U18 SN74CBTLV3245APW, U19 LME49721, U1X TPS562209SO, U2 AT93C46A-10TQ-2.7, U20 LME49721, U21 LME49721, U22 LME49721, U23 LME49721, U24 LMV358, U3X TPS3803-01DCKR, U4 TMS320C5535, U5 TMS320C5535, U6 FT2232HL, U7 TPD2E001IDRLRQ1, U8 74LVC1G175DBVSOT95, U9 W25Q64FVSFIG, U9-2 W25Q64FVSFIG, Y1 32.768kHz, Y1-2 32.768kHz

Commit message: 
Parts:
- C196: value 0.1u -> 2.2n
Changed lines of the file:
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@@
 <attribute name="MPN" value="2N7002ET1G" x="21.844" y="25.908" size="1.778" layer="27" rot="R270" display="off"/>
 </element>
-<element name="C196" library="SparkFun" package="0402-CAP" value="0.1u" x="31.242" y="29.21" rot="R180">
+<element name="C196" library="SparkFun" package="0402-CAP" value="2.2n" x="31.242" y="29.21" rot="R180">
 <attribute name="MPN" value="GRM155R71H222JA01J" x="31.242" y="29.21" size="1.778" layer="27" rot="R180" display="off"/>
 </element>
@@
 </signal>
 </signals>
-<errors>
-</errors>
 </board>
 </drawing>
