File: DMFX-2/DMFX-2 v1.0.brd (EAGLE design)
At the start: 100 x 68 mm, 56 parts, among them P5 87024-610LF, P7 87024-610LF, SW1X NAVIMEC

Commit message: 
Parts:
- VR5: value 50k -> 5k
Changed lines of the file:
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@@
 <attribute name="MPN" value="ERJ-2GE0R00X" x="77.502" y="9.201" size="1.778" layer="28" rot="MR270" display="off"/>
 </element>
-<element name="VR5" library="SparkFun" package="ALPS_POT" value="50k" x="73.912" y="34.028">
-<attribute name="MPN" value="EVU-F2AF30B54" x="73.912" y="34.028" size="1.778" layer="27" display="off"/>
+<element name="VR5" library="SparkFun" package="ALPS_POT" value="5k" x="73.912" y="34.028">
+<attribute name="MPN" value="EVU-F2AF30B53" x="73.912" y="34.028" size="1.778" layer="27" display="off"/>
 </element>
 <element name="D4X" library="led" package="LED3MM" value="RED" x="64.492" y="64.667">
@@
 </signal>
 </signals>
-<errors>
-</errors>
 </board>
 </drawing>
